File: pcb/expbox.sch (EAGLE design)
At the start: 48 parts, among them IC1 7805TV, K1 G5LE, Q1 2N3904, Q2 2N3904, Q3 2N3904, Q4 2N3904, Q5 2N3904, Q6 2N3904

Commit message: Replace buzzer with one with wider legs
Parts:
- removed SP1: KSS1201, buzzer:KSS1201
- added SG1: F/TMB, buzzer:F/TMB
Connections:
- net N$21: now also SG1.-; no longer SP1.2
- net VCC: now also SG1.+; no longer SP1.1
Changed lines of the file:
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@@
 <setting verticaltext="up"/>
 </settings>
-<grid distance="0.1" unitdist="inch" unit="inch" style="lines" multiple="1" display="yes" altdistance="0.01" altunitdist="inch" altunit="inch"/>
+<grid distance="0.1" unitdist="inch" unit="inch" style="lines" multiple="1" display="no" altdistance="0.01" altunitdist="inch" altunit="inch"/>
 <layers>
 <layer number="1" name="Top" color="4" fill="1" visible="no" active="no"/>
@@
 <part name="LED3" library="led" library_urn="urn:adsk.eagle:library:259" deviceset="LED" device="3MM" package3d_urn="urn:adsk.eagle:package:15797/1" value="red"/>
 <part name="R20" library="rcl" library_urn="urn:adsk.eagle:library:334" deviceset="R-EU_" device="R0805" package3d_urn="urn:adsk.eagle:package:23553/2" value="220"/>
-<part name="SP1" library="buzzer" library_urn="urn:adsk.eagle:library:113" deviceset="KSS1201" device="" package3d_urn="urn:adsk.eagle:package:5268/1"/>
 <part name="Q6" library="transistor-npn" library_urn="urn:adsk.eagle:library:398" deviceset="BC850*" device="SMD" package3d_urn="urn:adsk.eagle:package:28748/2" value="2N3904"/>
 <part name="GND16" library="supply1" library_urn="urn:adsk.eagle:library:371" deviceset="GND" device=""/>
@@
 <part name="U$3" library="abobija" deviceset="KCSA39-105" device=""/>
 <part name="U$4" library="abobija" deviceset="KCSA39-105" device=""/>
+<part name="SG1" library="buzzer" library_urn="urn:adsk.eagle:library:113" deviceset="F/TMB" device="" package3d_urn="urn:adsk.eagle:package:5260/1"/>
 </parts>
 <sheets>
@@
 <attribute name="VALUE" x="277.622" y="212.09" size="1.778" layer="96" rot="R90"/>
 </instance>
-<instance part="SP1" gate="1" x="434.34" y="236.22" smashed="yes" rot="R270">
-<attribute name="NAME" x="440.69" y="240.03" size="1.778" layer="95" rot="R270"/>
-<attribute name="VALUE" x="431.165" y="240.03" size="1.778" layer="96" rot="R270"/>
-</instance>
 <instance part="Q6" gate="G$1" x="431.8" y="213.36" smashed="yes">
 <attribute name="NAME" x="436.88" y="215.9" size="1.778" layer="95"/>
@@
 <attribute name="NAME" x="408.94" y="93.98" size="1.27" layer="95"/>
 <attribute name="VALUE" x="408.94" y="63.5" size="1.27" layer="96"/>
+</instance>
+<instance part="SG1" gate="1" x="436.88" y="238.76" smashed="yes" rot="R270">
+<attribute name="NAME" x="443.23" y="241.3" size="1.778" layer="95" rot="R270"/>
+<attribute name="VALUE" x="436.88" y="233.68" size="1.778" layer="96" rot="R270"/>
 </instance>
 </instances>
@@
 </segment>
 <segment>
-<pinref part="SP1" gate="1" pin="1"/>
 <pinref part="P+9" gate="VCC" pin="VCC"/>
 <wire x1="434.34" y1="241.3" x2="434.34" y2="251.46" width="0.1524" layer="91"/>
@@
 <wire x1="421.64" y1="251.46" x2="434.34" y2="251.46" width="0.1524" layer="91"/>
 <junction x="434.34" y="251.46"/>
+<pinref part="SG1" gate="1" pin="+"/>
 </segment>
 </net>
@@
 <segment>
 <pinref part="Q6" gate="G$1" pin="C"/>
-<pinref part="SP1" gate="1" pin="2"/>
 <wire x1="434.34" y1="218.44" x2="434.34" y2="220.98" width="0.1524" layer="91"/>
 <pinref part="D2" gate="G$1" pin="A"/>
-<wire x1="434.34" y1="220.98" x2="434.34" y2="231.14" width="0.1524" layer="91"/>
+<wire x1="434.34" y1="220.98" x2="434.34" y2="233.68" width="0.1524" layer="91"/>
 <wire x1="421.64" y1="223.52" x2="421.64" y2="220.98" width="0.1524" layer="91"/>
 <wire x1="421.64" y1="220.98" x2="434.34" y2="220.98" width="0.1524" layer="91"/>
 <junction x="434.34" y="220.98"/>
-</segment>
-</net>
+<pinref part="SG1" gate="1" pin="-"/>
+</segment>
+</net>
